File: PTP_project1/PTP_project1.kicad_sch (KiCad schematic)
At the start: 2 parts

Commit message: LV_2
Parts:
- added C1: 10u, symbol Device:C
- added C2: 100n, symbol Device:C
- added C3: 1u, symbol Device:C
- added C4: 22u, symbol Device:C_Polarized_Small
- added C5: 220u, symbol Device:C_Polarized_Small
- added D1: 11DQ06, Diode_SMD:D_SMA, symbol Diode:SS310
- added D2, D3, D4, D5: LED, symbol Device:LED
- added J1: Screw_Terminal_01x02, symbol Connector:Screw_Terminal_01x02
- added L1: 330u, symbol Device:L
- added R3, R4: 2k, symbol Device:R_Small
- added R5, R6, R7, R8: 4k7, symbol Device:R_Small
- added SW1: ~, symbol Switch:SW_MEC_5G
- added SW2: SW_SPDT_312, symbol Switch:SW_SPDT_312
- added U1: NE555P, Package_DIP:DIP-8_W7.62mm, symbol Timer:NE555P
- added U2: LM2574N-5, Package_DIP:DIP-8_W7.62mm, symbol Regulator_Switching:LM2574N-5
- R1, R2: value R_Small -> 47k
Connections:
- net GND: now also C1.2, C2.2, C3.1, C4.2, C5.2, D1.2 (A), J1.1 (Pin_1), R5.2, R6.2, R7.2, R8.2, SW1.1 (A), SW1.2 (A), U1.1 (GND), U2.2 (SGND), U2.3 (~{ON}/OFF), U2.4 (PGND); no longer R2.2
- net +3.3V renamed +5V
- net +5V: now also C2.1, C5.1, L1.2, R4.1, U1.4 (R), U1.8 (VCC), U2.1 (FB)
- net U_izl: no longer names the net of R1.2, R2.1
- net U_izl: now also U1.7 (DIS)
- new net: D2.1 (K), R5.1
- new net: D1.1 (K), L1.1, U2.7 (OUT)
- new net: D5.1 (K), R8.1
- new net: C1.1, R2.2, U1.2 (TR), U1.6 (THR)
- new net: D4.1 (K), R7.1
- new net: C3.2, R3.2, R4.2, SW2.3 (A)
- new net: R3.1, SW1.3 (B), SW1.4 (B)
- new net: D3.1 (K), R6.1
- new net 555: SW2.2 (C), U1.3 (Q)
- new net Q0: D2.2 (A)
- new net Q1: D3.2 (A)
- new net Q2: D4.2 (A)
- new net Q3: D5.2 (A)
- new net VD: C4.1, J1.2 (Pin_2), U2.5 (VIN)
- new net clock: SW2.1 (B)

Commit message: LV_3
Parts:
- added U6: SN74LVC1G11, SOT-23-6:SOT-23-6, symbol SN74LVC1G11:SN74LVC1G11
- R7: renamed from R4; value 2k -> 10K
- renumbered C4 to C1, C5 to C2, C2 to C4, C1 to C5, D2 to D1, D3 to D2, D4 to D3, D1 to D4, R5 to R1, R3 to R13, R1 to R19, R6 to R2, R2 to R20, R7 to R3, R8 to R4, U2 to U1, U1 to U7
Connections:
- net +5V: now also U6.5 (VCC)
- net GND: now also U6.2 (GND)
- net Q1: now also U6.1 (A)
- net Q3: now also U6.3 (B)
- net clock: now also R7.2
- net at C3.2, R13.2, SW2.3 (A): no longer R7.2
- new net Clock: U6.6 (C)
- new net Reset: U6.4 (Y)
Other:
- moved on the sheet: R7

Commit message: LV_4
Parts:
- added H1, H2, H3, H4: MountingHole, symbol Mechanical:MountingHole
- added R10, R11, R12, R9: 10k, symbol Device:R_Small
- added R14, R16, R17, R18, R5, R6, R8: 2k, symbol Device:R_Small
- added R15: R_Small, symbol Device:R_Small
- added U2, U3: 4027, symbol 4xxx:4027
- added U4: 74LS47, symbol 74xx:74LS47
- added U5: HDSP-7401, Display_7Segment:HDSP-7401, symbol Display_Character:HDSP-7401
- C1: footprint (none) -> Capacitor_THT:CP_Radial_D5.0mm_P2.00mm; Manufacturer (none) -> AISHI; Manufacturer Part Number  (none) -> EWH1EM220D11OT
- C2: footprint (none) -> Capacitor_THT:CP_Radial_D5.0mm_P2.00mm; Manufacturer (none) -> SAMWHA; Manufacturer Part Number  (none) -> RD1A227M05011BB
- D4: footprint Diode_SMD:D_SMA -> Diode_THT:D_DO-41_SOD81_P12.70mm_Horizontal; Manufacturer (none) -> SMC DIODE SOLUTIONS; Manufacturer Part Number  (none) -> 11DQ06TA
- J1: footprint (none) -> TerminalBlock_MetzConnect:TerminalBlock_MetzConnect_Type011_RT05502HBLC_1x02_P5.00mm_Horizontal; Manufacturer (none) -> DEGSON ELECTRONICS; Manufacturer Part Number  (none) -> DG301-5.0-02P-12-00A(H)
- U1: Manufacturer  (none) -> ONSEMI; Manufacturer Part Number (none) -> LM2574N-5G
- U6: footprint SOT-23-6:SOT-23-6 -> Package_TO_SOT_SMD:SOT-23-6; Manufacturer (none) -> TEXAS INSTRUMENTS; Manufacturer Part Number  (none) -> SN74LVC1G11DBVR
Connections:
- net clock is gone; now on net Clock: R7.2, SW2.1 (B)
- net +5V: now also R10.1, R11.1, R12.1, R15.1, R9.1, U2.16 (VDD), U3.16 (VDD), U4.16 (VCC), U5.1 (CA), U5.6 (CA)
- net Clock: now also U2.3 (C)
- net GND: now also U2.7 (S), U2.8 (VSS), U2.9 (S), U3.7 (S), U3.8 (VSS), U3.9 (S), U4.8 (GND)
- net Q0: now also U2.1 (Q), U2.13 (C), U4.7 (A)
- net Q1: now also U2.15 (Q), U3.3 (C), U4.1 (B)
- net Q2: now also U3.1 (Q), U3.13 (C), U4.2 (C)
- net Q3: now also U3.15 (Q), U4.6 (D)
- net Reset: now also U2.12 (R), U2.4 (R), U3.12 (R), U3.4 (R)
- new net: R14.1, U4.10 (d)
- new net: R8.1, U4.11 (c)
- new net: R6.1, U4.12 (b)
- new net: R5.1, U4.13 (a)
- new net: R18.1, U4.14 (g)
- new net: R17.1, U4.15 (f)
- new net: R15.2, U4.3 (LT), U4.4 (BI), U4.5 (RBI)
- new net: R16.1, U4.9 (e)
- new net: R9.2, U2.5 (K), U2.6 (J)
- new net: R11.2, U3.5 (K), U3.6 (J)
- new net: R14.2, U5.5 (D)
- new net: R18.2, U5.3 (G)
- new net: R12.2, U3.10 (J), U3.11 (K)
- new net: R8.2, U5.8 (C)
- new net: R10.2, U2.10 (J), U2.11 (K)
- new net: R16.2, U5.4 (E)
- new net: R6.2, U5.9 (B)
- new net: R5.2, U5.10 (A)
- new net: R17.2, U5.2 (F)
- no-connect marks 1 -> 6
Other:
- note added: "555 timer"
- note added: "JK vistabil"
- note added: "LED diode"
- note added: "Montažne rupe"
- note added: "Napajanje"
- note added: "Napajanje bistabila"
- note added: "Reset brojač"
- note added: "Tipkalo i ulaz radnog takta"
- moved on the sheet: C1, C2, D4, J1, L1, U1, U6

Commit message: domaca_zadaca
Parts:
- C3: footprint (none) -> Capacitor_SMD:C_1206_3216Metric_Pad1.33x1.80mm_HandSolder; Manufacturer (none) -> SAMSUNG; Manufacturer Part Number  (none) -> CL31B105KBHNNNE
- C4: footprint (none) -> Capacitor_SMD:C_1206_3216Metric_Pad1.33x1.80mm_HandSolder; Manufacturer (none) -> SAMSUNG; Manufacturer Part Number  (none) -> CL31B104KBCNNNC
- C5: footprint (none) -> Capacitor_SMD:C_1206_3216Metric_Pad1.33x1.80mm_HandSolder; Manufacturer (none) -> SAMSUNG; Manufacturer Part Number  (none) -> CL31A106KBHNNNE
- D1, D2, D3, D5: footprint (none) -> LED_THT:LED_D5.0mm
- H1, H2, H3, H4: footprint (none) -> MountingHole:MountingHole_5.5mm
- L1: footprint (none) -> Inductor_THT:L_Radial_D7.2mm_P3.00mm_Murata_1700; Manufacturer (none) -> FERROCORE; Manufacturer Part Number  (none) -> COIL0608-0.33
- R1, R2, R3, R4: footprint (none) -> Resistor_THT:R_Axial_DIN0207_L6.3mm_D2.5mm_P10.16mm_Horizontal
- R10, R11, R12, R7, R9: footprint (none) -> Resistor_SMD:R_1206_3216Metric_Pad1.30x1.75mm_HandSolder
- R13, R14, R16, R17, R18, R5, R6, R8: footprint (none) -> Resistor_SMD:R_1206_3216Metric_Pad1.30x1.75mm_HandSolder; Manufacturer (none) -> ROYALOHM; Manufacturer Part Number  (none) -> 1206S4F2001T5E
- R15: value R_Small -> 10k; footprint (none) -> Resistor_SMD:R_1206_3216Metric_Pad1.30x1.75mm_HandSolder
- R19, R20: footprint (none) -> Resistor_SMD:R_1206_3216Metric_Pad1.30x1.75mm_HandSolder; Manufacturer (none) -> ROYALOHM; Manufacturer Part Number  (none) -> 1206S4J0473T5E
- SW1: footprint (none) -> Button_Switch_THT:SW_PUSH_6mm_H4.3mm; Manufacturer (none) -> microswitch TACT; Manufacturer Part Number  (none) -> TACT-64N-F
- SW2: footprint (none) -> Button_Switch_THT:SW_Slide_SPDT_Straight_CK_OS102011MS2Q; Manufacturer (none) -> C&K; Manufacturer Part Number (none) -> OS102011MS2QN1C
- U2, U3: footprint (none) -> Package_DIP:DIP-16_W7.62mm_Socket_LongPads; Manufacturer (none) -> RENESAS; Manufacturer Part Number  (none) -> CD4027BMS
- U4: footprint (none) -> Package_DIP:DIP-16_W7.62mm_Socket_LongPads; Manufacturer (none) -> TEXAS INSTRUMENTS; Manufacturer Part Number  (none) -> SN74LS47N
- U5: Manufacturer (none) -> FORYARD; Manufacturer Part Number  (none) -> FYS-3911BUHR-21
- U7: Manufacturer (none) -> TEXAS INSTRUMENTS; Manufacturer Part Number  (none) -> NE555P
